Commit message: Important cosmetic changes for more clarity and update to viewer

File: urdf/obstacles.urdf (robot description, URDF)
Before this commit: robot obstacles, 2 links, 1 joints
Links:
- link l_object_one: geometry collision cylinder length=2. radius=0.07; visual cylinder length=2. radius=0.07
- link obstacle_base: geometry collision cylinder length=2. radius=0.07; visual cylinder length=2. radius=0.07
