Commit message: Add lights and longer bar, update to new optimizer (icra2016)

File: urdf/ur5_robot.urdf (robot description, URDF)
Before this commit: robot ur5, 8 links, 7 joints
Links:
- link ee_link: geometry collision cylinder length=0.2 radius=0.01; visual cylinder length=0.2 radius=0.01
Joints:
- joint ee_fixed_joint: origin xyz=0.0 0.13 0.0 rpy=1.570796325 0.0 0.0 -> xyz=0.0 0.18 0.0 rpy=1.570796325 0.0 0.0
