Commit message: Use visual meshes for collision, Add sphere obstacles problem

File: urdf/obstacle_sphere.urdf (robot description, URDF)
Before this commit: robot obstacles, 2 links, 1 joints
Links:
- link l_object_one: geometry collision sphere radius=0.2; visual sphere radius=0.2
- link obstacle_base: geometry collision sphere radius=0.2; visual sphere radius=0.2

Commit message: Fix UR5 bugs and update scripts:
* ? fix UR5 meshes
* add FIAD ur5-with-gripper, carton, box files
* add trajectory plot functions
* update script to TADR2, add convergence graphs

File: urdf/obstacle_sphere.urdf (robot description, URDF)
Before this commit: robot obstacles, 2 links, 1 joints
Links:
- link l_object_one: geometry collision mesh filename=package://ur_description/meshes/sphere.dae scale=0.18 0.18 0.18; visual sphere radius=0.18
- link obstacle_base: geometry collision mesh filename=package://ur_description/meshes/sphere.dae scale=0.18 0.18 0.18; visual sphere radius=0.18

File: urdf/obstacles.urdf (robot description, URDF)
Before this commit: robot obstacles, 2 links, 1 joints
Links:
- link l_object_one: geometry collision mesh filename=package://ur_description/meshes/cylinder.dae; visual cylinder length=2. radius=0.07
- link obstacle_base: geometry collision mesh filename=package://ur_description/meshes/cylinder.dae; visual cylinder length=2. radius=0.07

File: urdf/ur5_with_gripper.urdf (robot description, URDF)
Before this commit: robot ur5, 8 links, 7 joints
Links:
- removed link ee_link
- added link gripper_link; collision mesh filename=package://ur_description/meshes/gripper.dae; visual mesh filename=package://ur_description/meshes/gripper.dae
Joints:
- joint ee_fixed_joint: child ee_link -> gripper_link; origin xyz=0.0 0.18 0.0 rpy=1.570796325 0.0 0.0 -> xyz=0.0 0.0 0.0 rpy=1.570796325 0.0 0.0
